Commit message: camera fix orientation and position

File: realsense2_description/urdf/_d455.urdf.xacro (robot description, xacro)
@@ -2,7 +2,7 @@
 <robot name="sensor_d455" xmlns:xacro="http://ros.org/wiki/xacro">
   <xacro:include filename="$(find realsense2_description)/urdf/_materials.urdf.xacro" />
-  <!-- TODO: investigate what this is for -->
+  <!-- TODO investigate what this is for -->
   <!-- <xacro:include filename="$(find realsense2_description)/urdf/_usb_plug.urdf.xacro" /> -->
-  <xacro:macro name="sensor_d455" params="parent *origin name:=camera use_nominal_extrinsics:=false">
+  <xacro:macro name="sensor_d455" params="parent *origin name:=camera_01 use_nominal_extrinsics:=false">
     <xacro:arg name="add_plug" default="false" />
     <xacro:property name="M_PI" value="3.1415926535897931" />
@@ -23,4 +23,7 @@
     <xacro:property name="d455_cam_depth_py" value="0.0475"/>
     <xacro:property name="d455_cam_depth_pz" value="${d455_cam_height/2}"/>
+    <!-- The following values model camera's plugin orientation -->
+    <xacro:property name="d455_cam_R" value="1.57"/>
+    <xacro:property name="d455_cam_P" value="-1.57"/>
     <!-- camera body, with origin at bottom screw mount -->
     <joint name="${name}_joint" type="fixed">
@@ -156,5 +159,5 @@
     <gazebo reference="${name}_depth_optical_frame">
         <sensor name="cameradepth" type="depth_camera">
-            <pose>0 0 0 0 0 0</pose>
+            <pose>0 0 0 ${d455_cam_R} ${d455_cam_P} 0.0</pose>
             <camera name="camera">
                 <horizontal_fov>1.518</horizontal_fov> <!-- 87 degrees for depth -->
@@ -177,5 +180,5 @@
     <gazebo reference="${name}_color_optical_frame">
         <sensor name="cameracolor" type="camera">
-            <pose>0 0 0 0 0 0</pose>
+            <pose>0 0 0 ${d455_cam_R} ${d455_cam_P} 0.0</pose>
             <camera name="camera">
                 <horizontal_fov>1.518</horizontal_fov> <!-- 87 degrees for depth -->
@@ -204,4 +207,5 @@
     <gazebo reference="${name}_infra1_optical_frame">
         <sensor name="cameraired1" type="camera">
+        <pose>0 0 0 ${d455_cam_R} ${d455_cam_P} 0.0</pose>
         <camera name="camera">
             <horizontal_fov>1.57</horizontal_fov>
@@ -230,4 +234,5 @@
     <gazebo reference="${name}_infra2_optical_frame">
         <sensor name="cameraired2" type="camera">
+        <pose>0 0 0 ${d455_cam_R} ${d455_cam_P} 0.0</pose>
             <camera name="camera">
                 <horizontal_fov>1.57</horizontal_fov>

File: realsense2_description/urdf/test_d455_camera.urdf.xacro (robot description, xacro)
@@ -3,6 +3,10 @@
   <xacro:arg name="use_nominal_extrinsics" default="true"/>
   <xacro:include filename="$(find realsense2_description)/urdf/_d455.urdf.xacro" />
-  <link name="base_link" />
-  <xacro:sensor_d455 parent="base_link" use_nominal_extrinsics="$(arg use_nominal_extrinsics)">
+  <link name="world"/>
+  <gazebo reference="world">
+      <static>true</static>
+  </gazebo>
+  <!-- <link name="base_link" /> -->
+  <xacro:sensor_d455 parent="world" use_nominal_extrinsics="$(arg use_nominal_extrinsics)">
     <origin xyz="0 0 0" rpy="0 0 0"/>
   </xacro:sensor_d455>

Commit message: fixes following the tf tree fix. potential for reviews

File: realsense2_description/urdf/_d455.urdf.xacro (robot description, xacro)
@@ -168,5 +168,5 @@
                 <clip>
                     <near>0.1</near>
-                    <far>100.0</far>
+                    <far>5.0</far>
                 </clip>
             </camera>
@@ -174,5 +174,5 @@
             <update_rate>30</update_rate>
             <visualize>true</visualize>
-            <gz_frame_id>${name}_depth_optical_frame</gz_frame_id>
+            <gz_frame_id>${name}_depth_frame</gz_frame_id>
             <topic>${name}/camera_depth</topic>
         </sensor>
@@ -261,9 +261,9 @@
     <gazebo>
         <plugin filename="ignition-gazebo-pose-publisher-system" name="gz::sim::systems::PosePublisher">
-            <publish_link_pose>true</publish_link_pose>
+            <publish_link_pose>false</publish_link_pose>
             <publish_visual_pose>false</publish_visual_pose>
             <publish_collision_pose>false</publish_collision_pose>
             <publish_sensor_pose>false</publish_sensor_pose>
-            <publish_model_pose>false</publish_model_pose>
+            <publish_model_pose>true</publish_model_pose>
             <publish_nested_model_pose>true</publish_nested_model_pose>
             <use_pose_vector_msg>true</use_pose_vector_msg>

File: realsense2_description/urdf/test_d455_camera.urdf.xacro (robot description, xacro)
@@ -3,11 +3,11 @@
   <xacro:arg name="use_nominal_extrinsics" default="true"/>
   <xacro:include filename="$(find realsense2_description)/urdf/_d455.urdf.xacro" />
-  <link name="world"/>
-  <gazebo reference="world">
+  <link name="realsense2_camera"/>
+  <!-- <link name="base_link" /> -->
+  <xacro:sensor_d455 parent="realsense2_camera" use_nominal_extrinsics="$(arg use_nominal_extrinsics)">
+    <origin xyz="0 0 0" rpy="0 0 0"/>
+  </xacro:sensor_d455>
+  <gazebo>
       <static>true</static>
   </gazebo>
-  <!-- <link name="base_link" /> -->
-  <xacro:sensor_d455 parent="world" use_nominal_extrinsics="$(arg use_nominal_extrinsics)">
-    <origin xyz="0 0 0" rpy="0 0 0"/>
-  </xacro:sensor_d455>
 </robot>
